File: 258Verbos.kicad_pcb (KiCad board)
At the start: 2 copper layers, 79.9 x 106.7 mm, 154 parts, among them IC1 CA3140N, IC2 CA3140N, J1 J201, J2 J201, Q1 2N3906, Q2 BC847BS, Q3 J113, Q4 2N3906, Q5 BC847BS, Q6 J113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

Commit message: Modified footprint for pots. Changed silkscreen text. Rerouted
Parts:
- 10R1: value 0.5W -> 10R
- IC2: value CA3140N -> CA3140
Routing:
- net +15V: track 0.00 -> 389.8 mm, vias 0 -> 7
- net -15V: track 0.00 -> 297.5 mm, vias 0 -> 10
- net /N$38: track 0.00 -> 122.1 mm, vias 0 -> 4
- net Net-(C7-Pad2): track 0.00 -> 111.7 mm, vias 0 -> 1
- net Net-(C10-Pad1): track 0.00 -> 111.3 mm, vias 0 -> 2
- net Net-(C9-Pad1): track 0.00 -> 108.4 mm, vias 0 -> 3
- net Net-(R58-Pad2): track 0.00 -> 108.2 mm
- net /N$43: track 0.00 -> 106.5 mm, vias 0 -> 2
- net Net-(CONTROL1-Pad3): track 0.00 -> 99.5 mm, vias 0 -> 2
- net Net-(R15-Pad1): track 0.00 -> 96.9 mm, vias 0 -> 2
- net /N$18: track 0.00 -> 93.8 mm, vias 0 -> 3
- net Net-(R64-Pad2): track 0.00 -> 88.3 mm, vias 0 -> 4
- net Net-(Q6-Pad1): track 0.00 -> 87.5 mm, vias 0 -> 2
- net Net-(R82-Pad2): track 0.00 -> 84.4 mm, vias 0 -> 1
- net /N$12: track 0.00 -> 81.2 mm, vias 0 -> 3
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Other:
- board text added: "BES 004:- Dual Analogue VCO Rev: 2.1"
- board text added: "Barry Synnott Feb 2018"
- board text added: "Box Emissions Systems"
- board text added: "O1 Sine Adj"
- board text added: "O1 V/Oct"
- board text added: "O2 Sine Adj"
- board text added: "O2 V/Oct"
- board text added: "V/Oct"
- board text removed: "BES 004:- Dual Analogue VCO Rev: 2"
- board text removed: "Barry Synnott Feb 2017"
- board text removed: "O1 Sine"
- board text removed: "O1 V"
- board text removed: "O2 Sine"
- board text removed: "O2 V"
